File: design_project.kicad_pcb (KiCad board)
At the start: 2 copper layers, 82 x 62.7 mm, 55 parts, among them J1 Conn_01x02, J2 Conn_02x16_Top_Bottom, J3 USB_C_Receptacle_PowerOnly_6P, Q1 AO3401CI-ES, Q3 2N7002, SW1 SW_Wuerth_450301014042, U1 INA219AIDCNR, U10 AP22804AW5, U2 DRV8833PWP, U3 DRV8833PWP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

Commit message: 2nd round
Co-Authored-By: Thaboish565 <176961582+thaboish565@users.noreply.github.com>
Parts:
- moved U1 7.93 mm to (148.5, 83.5)
- moved U6 4.83 mm to (132.0, 111.0)
- moved U5 4.31 mm to (139.4, 103.8)
- moved SW1 4.31 mm to (124.8, 106.3)
- moved U4 2.35 mm to (146.5, 91.5)
- turned U6 to -90 degrees
- turned U7 to 180 degrees
Routing:
- net Net-(Q3-D): track 0.00 -> 98.3 mm, vias 0 -> 1
- net I2C1_SDA: track 61.1 -> 151.6 mm
- net 5V: track 70.7 -> 149.7 mm, vias 0 -> 3
- net Net-(U3-AISEN): track 0.00 -> 76.0 mm, vias 0 -> 5
- net High Voltage (9V): track 10.2 -> 75.9 mm, vias 0 -> 2
- net 3.3V: track 60.3 -> 118.0 mm
- net Net-(U3-BISEN): track 77.4 -> 121.3 mm
- net Net-(U6-BAT): track 31.7 -> 68.7 mm
- net Battery: track 30.5 -> 53.0 mm
- net Net-(U1-IN-): track 0.00 -> 21.2 mm, vias 0 -> 1
- net Net-(U9-SW): track 0.00 -> 16.3 mm, vias 0 -> 1
- net Net-(U1-IN+): track 16.4 -> 27.5 mm, vias 0 -> 1
- net MOTOR2_A_OUT: track 11.1 -> 22.0 mm
- net MOTOR1_B_OUT: track 19.3 -> 28.3 mm, vias 0 -> 3
- net CTRL_EXT_LOAD1 : track 96.4 -> 105.3 mm
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- added copper zone on F.Cu, net (none)
